Commit message: Added RPlidar and ZED Urdf Links and Joints

File: urdf/jeep.urdf (robot description, URDF)
Before this commit: robot jeepModel, 6 links, 5 joints
Links:
- added link laser_base_link; visual mesh filename=package://ros_robotics/meshes/RpLidarBase.stl scale=0.001 0.001 0.001
- added link laser_spinny_link; visual mesh filename=package://ros_robotics/meshes/RpLidarSpinnyTop.stl scale=0.001 0.001 0.001
- added link zed_camera_center; visual mesh filename=package://ros_robotics/meshes/zed.stl
- added link zed_left_camera_frame
- added link zed_left_camera_optical_frame
- added link zed_right_camera_frame
- added link zed_right_camera_optical_frame
Joints:
- added joint ZED_right_camera_joint: type fixed, parent zed_camera_center, child zed_right_camera_frame, origin xyz=0 -0.03 0 rpy=0 0 0
- added joint base_link_to_ZED_camera_center: type fixed, parent base_link, child zed_camera_center, origin xyz=0.095 0 0.577 rpy=0 0 0
- added joint base_link_to_lidar_base: type fixed, parent base_link, child laser_base_link, origin xyz=0.0152 -0.004 0.56 rpy=0 0 0
- added joint base_link_to_zed_left_optical: type fixed, parent base_link, child zed_left_camera_optical_frame, origin xyz=0 0 0 rpy=-1.57079632679 0.0 -1.57079632679
- added joint lidar_base_to_spinny_link: type continuous, parent laser_base_link, child laser_spinny_link, origin xyz=0.0179 0.001 0.0465 rpy=0 0 0
- added joint zed_left_camera_joint: type fixed, parent zed_camera_center, child zed_left_camera_frame, origin xyz=0 0.03 0 rpy=0 0 0
- added joint zed_left_camera_optical_joint: type fixed, parent zed_left_camera_frame, child zed_left_camera_optical_frame, origin xyz=0 0 0 rpy=-1.57079632679 0.0 -1.57079632679
- added joint zed_right_camera_optical_joint: type fixed, parent zed_right_camera_frame, child zed_right_camera_optical_frame, origin xyz=0 0 0 rpy=-1.57079632679 0.0 -1.57079632679

Commit message: Removed Sensor Platform Link and Joint
Sensor Platform Link and Joint deemed unnecessary for urdf configuration. Only added unnecessary work

File: urdf/jeep.urdf (robot description, URDF)
Before this commit: robot jeepModel, 13 links, 13 joints
Links:
- removed link sensor_platform
Joints:
- removed joint sensor_platform_to_base_link

Commit message: Added HTC Vive Tracker support

File: urdf/jeep.urdf (robot description, URDF)
Before this commit: robot jeepModel, 12 links, 12 joints
Links:
- added link Base_Frame; visual mesh filename=package://ros_robotics/meshes/LILBOT_w_wheels.xml scale=0.001 0.001 0.001
- added link Lighthouse BeFrame; visual box size=0.1 0.1 0.1
- added link Lighthouse Frame; visual box size=0.05 0.05 0.05
- added link base_footprint
- added link laser_data_link; visual box size=0.02 0.02 0.02
- added link lighthouse_mount; visual box size=0.05 0.05 0.05
- added link lighthouse_rotate; visual box size=0.05 0.05 0.05
- added link maximum_lighthouse_x; visual box size=0.05 4.05 0.05
- added link maximum_lighthouse_xy; visual box size=2.65 0.05 0.05
- added link minimum_lighthouse_x; visual box size=0.05 4.05 0.05
- added link minimum_lighthouse_xy; visual box size=2.65 0.05 0.05
Joints:
- added joint Base_footprint_to_libot_base: type fixed, parent base_footprint, child Base_Frame, origin xyz=0 0 0.160 rpy=0 0 0
- added joint base_footprint_to_base_link: type fixed, parent base_footprint, child base_link, origin xyz=0 0 0.160 rpy=0 0 0
- added joint base_link_to_maximum_lighthouse_x: type fixed, parent base_link, child maximum_lighthouse_x, origin xyz=4.0 0 0 rpy=0 0 0
- added joint base_link_to_maximum_lighthouse_xy: type fixed, parent base_link, child maximum_lighthouse_xy, origin xyz=2.7 2 0 rpy=0 0 0
- added joint base_link_to_minimum_lighthouse_x: type fixed, parent base_link, child minimum_lighthouse_x, origin xyz=1.4 0 0 rpy=0 0 0
- added joint base_link_to_minimum_lighthouse_xy: type fixed, parent base_link, child minimum_lighthouse_xy, origin xyz=2.7 -2 0 rpy=0 0 0
- added joint laser_base_link_to_data_link: type fixed, parent laser_base_link, child laser_data_link, origin xyz=0.02 0 0.0415 rpy=0 0 0
- added joint laser_data_to_base_link: type fixed, parent base_link, child laser_data_link, origin xyz=0.02 0 0.6 rpy=0 0 0
- added joint lighthouse_beframe_to_lighthouse_frame: type fixed, parent Lighthouse BeFrame, child Lighthouse Frame, origin xyz=0 0 0.1002 rpy=0 0 0.0
- added joint lighthouse_mount_to_lighthouse_rotate: type fixed, parent lighthouse_mount, child lighthouse_rotate, origin xyz=0 0 0.57 rpy=0.43 0.03 0
- added joint lighthouse_rotate_to_lighthouse_beframe: type fixed, parent lighthouse_rotate, child Lighthouse BeFrame, origin xyz=0 0 0.07620 rpy=1.57079632679 3.14159 0.0
- added joint sensor_platform_to_lighthouse_mount: type fixed, parent base_link, child lighthouse_mount, origin xyz=0.85 0 0.0 rpy=0 0 1.57079632679
